File: aom_driver.kicad_pcb (KiCad board)
At the start: 4 copper layers, 165.1 x 76.2 mm, 154 parts, among them J1 Conn_Coaxial, J2 Conn_Coaxial, J3 Screw_Terminal_01x03, U1 LT3082xDD, U10 RVA-3000R, U11 ADP7182AUJZ-5.0, U12 M3SWA-2-50, U13 LT3082xDD, U14 LT3082xDD, U15 LT3082xDD, U16 PAT1220-C-8DB, U17 LT3082xDD, U18 GVA-81, U19 RVA-3000R, U2 ADP7182AUJZ-5.0, U20 ADP7182AUJZ-5.0, U21 M3SWA-2-50, U3 M3SWA-2-50, U4 LT3082xDD, U5 LT3082xDD, U6 LT3082xDD, U7 PAT1220-C-8DB, U8 LT3082xDD, U9 GVA-81, X1 CVCO55xx, X2 CVCO55xx

Commit message: v2
Parts:
- removed the C24 at (108.6, 71.1)
- removed the C43 at (108.6, 103.1)
- removed the L1 at (108.7, 95.9)
- removed L3, L4, L6: 10u, Inductor_SMD:L_0805_2012Metric_Pad1.05x1.20mm_HandSolder
- removed REF**: OSHW-Logo2_9.8x8mm_SilkScreen, Symbol:OSHW-Logo2_9.8x8mm_SilkScreen
- removed REF**: KiCad-Logo2_5mm_SilkScreen, Symbol:KiCad-Logo2_5mm_SilkScreen
- removed the RV1 at (205.6, 85.1)
- removed RV3: 2M, Potentiometer_THT:Potentiometer_Bourns_3296Y_Vertical
- added C10: 0.1u, Capacitor_SMD:C_0805_2012Metric_Pad1.18x1.45mm_HandSolder, F.Cu at (187.5, 93.0)
- added C19: 0.1u, Capacitor_SMD:C_0805_2012Metric_Pad1.18x1.45mm_HandSolder, F.Cu at (147.8, 124.6)
- added C21: 0.1u, Capacitor_SMD:C_0805_2012Metric_Pad1.18x1.45mm_HandSolder, F.Cu at (147.8, 92.6)
- added C25: 0.1u, Capacitor_SMD:C_0805_2012Metric_Pad1.18x1.45mm_HandSolder, F.Cu at (164.7, 122.3)
- added C26: 0.1u, Capacitor_SMD:C_0805_2012Metric_Pad1.18x1.45mm_HandSolder, F.Cu at (164.7, 90.3)
- added C37: 0.1u, Capacitor_SMD:C_0805_2012Metric_Pad1.18x1.45mm_HandSolder, F.Cu at (124.8, 122.4)
- added C38: 0.1u, Capacitor_SMD:C_0805_2012Metric_Pad1.18x1.45mm_HandSolder, F.Cu at (124.8, 90.4)
- added C51: 0.1u, Capacitor_SMD:C_0805_2012Metric_Pad1.18x1.45mm_HandSolder, F.Cu at (91.4, 104.3)
- added C52: 0.1u, Capacitor_SMD:C_0805_2012Metric_Pad1.18x1.45mm_HandSolder, F.Cu at (95.6, 130.8)
- added C55: 2.2u, Capacitor_SMD:C_0805_2012Metric_Pad1.18x1.45mm_HandSolder, F.Cu at (81.0, 117.3)
- added C7: 0.1u, Capacitor_SMD:C_0805_2012Metric_Pad1.18x1.45mm_HandSolder, F.Cu at (205.5, 116.3)
- added C8: 0.1u, Capacitor_SMD:C_0805_2012Metric_Pad1.18x1.45mm_HandSolder, F.Cu at (205.6, 84.3)
- added C9: 0.1u, Capacitor_SMD:C_0805_2012Metric_Pad1.18x1.45mm_HandSolder, F.Cu at (187.5, 125.0)
- added R1: 0, Resistor_SMD:R_0805_2012Metric_Pad1.20x1.40mm_HandSolder, F.Cu at (209.4, 115.4)
- added R13: 1.5k, Resistor_SMD:R_0805_2012Metric_Pad1.20x1.40mm_HandSolder, F.Cu at (199.6, 110.7)
- added R14: 1.5k, Resistor_SMD:R_0805_2012Metric_Pad1.20x1.40mm_HandSolder, F.Cu at (199.6, 78.7)
- added R15: 1.5k, Resistor_SMD:R_0805_2012Metric_Pad1.20x1.40mm_HandSolder, F.Cu at (192.3, 120.0)
- added R16: 1.5k, Resistor_SMD:R_0805_2012Metric_Pad1.20x1.40mm_HandSolder, F.Cu at (192.3, 88.0)
- added R17: 0, Resistor_SMD:R_0805_2012Metric_Pad1.20x1.40mm_HandSolder, F.Cu at (148.8, 129.3)
- added R18: 0, Resistor_SMD:R_0805_2012Metric_Pad1.20x1.40mm_HandSolder, F.Cu at (148.8, 97.3)
- added R19: 0, Resistor_SMD:R_0805_2012Metric_Pad1.20x1.40mm_HandSolder, F.Cu at (172.2, 128.0)
- added R2: 0, Resistor_SMD:R_0805_2012Metric_Pad1.20x1.40mm_HandSolder, F.Cu at (209.3, 83.3)
- added R20: 0, Resistor_SMD:R_0805_2012Metric_Pad1.20x1.40mm_HandSolder, F.Cu at (172.2, 96.0)
- added R27: 1.5k, Resistor_SMD:R_0805_2012Metric_Pad1.20x1.40mm_HandSolder, F.Cu at (155.8, 123.3)
- added R28: 1.5k, Resistor_SMD:R_0805_2012Metric_Pad1.20x1.40mm_HandSolder, F.Cu at (155.8, 91.3)
- added R3: 0, Resistor_SMD:R_0805_2012Metric_Pad1.20x1.40mm_HandSolder, F.Cu at (194.6, 129.3)
- added R31: 1.5k, Resistor_SMD:R_0805_2012Metric_Pad1.20x1.40mm_HandSolder, F.Cu at (169.8, 118.5)
- added R32: 1.5k, Resistor_SMD:R_0805_2012Metric_Pad1.20x1.40mm_HandSolder, F.Cu at (169.8, 86.5)
- added R33: 0, Resistor_SMD:R_0805_2012Metric_Pad1.20x1.40mm_HandSolder, F.Cu at (119.0, 124.8)
- added R34: 0, Resistor_SMD:R_0805_2012Metric_Pad1.20x1.40mm_HandSolder, F.Cu at (119.0, 92.8)
- added R4: 0, Resistor_SMD:R_0805_2012Metric_Pad1.20x1.40mm_HandSolder, F.Cu at (194.6, 97.3)
- added R42: 0, Resistor_SMD:R_0805_2012Metric_Pad1.20x1.40mm_HandSolder, F.Cu at (109.7, 104.3)
- added R44: 0, Resistor_SMD:R_0805_2012Metric_Pad1.20x1.40mm_HandSolder, F.Cu at (109.7, 72.3)
- added R45: 1.5k, Resistor_SMD:R_0805_2012Metric_Pad1.20x1.40mm_HandSolder, F.Cu at (88.4, 109.4)
- added R54: 0, Resistor_SMD:R_0805_2012Metric_Pad1.20x1.40mm_HandSolder, F.Cu at (84.2, 99.6)
- added R55: 0, Resistor_SMD:R_0805_2012Metric_Pad1.20x1.40mm_HandSolder, F.Cu at (90.6, 133.2)
- added R6: 49.9k, Resistor_SMD:R_0805_2012Metric_Pad1.20x1.40mm_HandSolder, F.Cu at (200.4, 116.3)
- added R8: 0, Resistor_SMD:R_0805_2012Metric_Pad1.20x1.40mm_HandSolder, F.Cu at (200.7, 84.3)
- added SYM1: Logo_Open_Hardware_Small, Symbol:OSHW-Logo2_9.8x8mm_SilkScreen, F.Cu at (223.8, 109.9)
- added SYM2: Logo_Open_Hardware_Small, Symbol:KiCad-Logo2_5mm_SilkScreen, F.Cu at (223.8, 120.7)
- FL1: renamed from FL2; value RLP-158 -> RLP-320+
- R11: renamed from R22; value 432 -> 4.7k
- R12: renamed from R11; value 432 -> 4.7k
- R25: renamed from R24; value 432 -> 4.7k
- R26: renamed from R13; value 432 -> 4.7k
- R39: renamed from R29; value 432 -> 4.7k
- R40: renamed from R18; value 432 -> 4.7k
- R46: renamed from R5; value 432 -> 4.7k
- R47: renamed from R4; value 432 -> 4.7k
- R48: renamed from R7; value 2.43k -> 27k
- R49: renamed from R8; value 2.43k -> 27k
- R5: renamed from R20; value 2.7M -> 10M
- R7: renamed from R9; value 2.7M -> 150k
- RV1: renamed from RV4; footprint Potentiometer_THT:Potentiometer_Bourns_3296Y_Vertical -> Potentiometer_THT:Potentiometer_Bourns_3296X_Horizontal
- RV2: footprint Potentiometer_THT:Potentiometer_Bourns_3296Y_Vertical -> Potentiometer_THT:Potentiometer_Bourns_3296X_Horizontal
- moved RV1 48.9 mm to (114.0, 127.4)
- moved RV2 48.9 mm to (114.0, 95.4)
- moved C2 25.1 mm to (137.3, 97.3)
- moved C1 25.1 mm to (137.3, 129.3)
- moved R41 8.32 mm to (121.0, 78.9), turned to 0 degrees
- moved D10 5.85 mm to (91.2, 93.5), turned to 90 degrees
- moved D9 5.30 mm to (90.6, 76.8), turned to 90 degrees
- moved TP11 5.23 mm to (171.6, 115.7)
- moved TP12 5.23 mm to (171.6, 83.7)
- moved R35 4.49 mm to (124.8, 117.7)
- moved R37 4.49 mm to (124.8, 119.9)
- moved R36 4.49 mm to (124.8, 85.7)
- moved R38 4.49 mm to (124.8, 87.9)
- moved C15 3.74 mm to (152.9, 129.3), turned to 0 degrees
- moved C16 3.74 mm to (152.9, 97.3), turned to 0 degrees
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- renumbered C26 to C1, C29 to C11, C30 to C12, C10 to C13, C11 to C14, C31 to C15, C12 to C16, C33 to C17, C14 to C18, C7 to C2, C32 to C20, C13 to C22, C34 to C23, C15 to C24, C35 to C27, C16 to C28, C36 to C29, C27 to C3, C17 to C30, C37 to C31, C18 to C32, C38 to C33, C19 to C34, C39 to C35, C20 to C36, C40 to C39, C8 to C4, C21 to C40, C22 to C42, C42 to C43, C23 to C44, C44 to C45, C25 to C46, C3 to C47, C4 to C48, C6 to C49, C28 to C5, C5 to C50, C2 to C53, C1 to C54, C9 to C6, D8 to D1, D4 to D10, D5 to D2, D9 to D3, D6 to D4, D10 to D5, D7 to D6, D2 to D7, D1 to D8, D3 to D9, FL1 to FL2, L5 to L1, R23 to R21, R12 to R22, R25 to R23, R14 to R24, R26 to R29, R15 to R30, R27 to R35, R16 to R36, R28 to R37, R17 to R38, R19 to R41, R30 to R43, R6 to R50, R2 to R51, R3 to R52, R1 to R53, R21 to R9, TP16 to TP1, TP9 to TP10, TP21 to TP11, TP10 to TP12, TP22 to TP13, TP11 to TP14, TP23 to TP15, TP12 to TP16, TP24 to TP17, TP13 to TP18, TP14 to TP19, TP5 to TP2, TP25 to TP20, TP26 to TP21, TP15 to TP22, TP3 to TP23, TP4 to TP24, TP2 to TP25, TP1 to TP26, TP17 to TP3, TP6 to TP4, TP18 to TP5, TP7 to TP6, TP19 to TP7, TP20 to TP9, U13 to U1, U8 to U10, U18 to U11, U9 to U12, U19 to U13, U10 to U14, U20 to U15, U11 to U16, U21 to U17, U12 to U18, U3 to U19, U14 to U2, U2 to U20, U1 to U21, U4 to U3, U5 to U4, U15 to U5, U16 to U7, U7 to U8, U17 to U9, X2 to X1, X1 to X2
Connections:
- net /F1/+5V renamed /+5V_CH2
- net /F1/-5V renamed /-5V_CH2
- net /F1/F_OUT renamed Net-(U18-RF-IN)
- net /F1/VCO_TUNE renamed /VCO_TUNE_CH2
- net /F1/VDD_VCO renamed /VDD_VCO_CH2
- net /F1/VVA_TUNE renamed /VVA_TUNE_CH2
- net /F2/+5V renamed /+5V_CH1
- net /F2/-5V renamed /-5V_CH1
- net /F2/F_OUT renamed Net-(U17-RF-IN)
- net /F2/VCO_TUNE renamed /VCO_TUNE_CH1
- net /F2/VDD_VCO renamed /VDD_VCO_CH1
- net /F2/VVA_TUNE renamed /VVA_TUNE_CH1
- net SW renamed Net-(J2-In)
- C15 pad 1: Net-(C27-Pad1) (its old number) -> Net-(C15-Pad1)
- C16 pad 1: Net-(C12-Pad1) -> Net-(C16-Pad1)
- C17 pad 1: Net-(C27-Pad1) (its old number) -> Net-(C17-Pad1)
- C18 pad 1: Net-(C12-Pad1) -> Net-(C18-Pad1)
- C3 pad 1: Net-(C27-Pad1) (its old number) -> Net-(C3-Pad1)
- C35 pad 2: VEE -> Net-(U15-VIN)
- C36 pad 2: VEE -> Net-(U16-VIN)
- C4 pad 1: Net-(C12-Pad1) -> Net-(C4-Pad1)
- C44 pad 2: Net-(U12-RF-OUT1) -> Net-(U18-RF-OUT2)
- C5 pad 1: Net-(C27-Pad1) (its old number) -> Net-(C5-Pad1)
- C53 pad 1: VDD -> Net-(C53-Pad1)
- C54 pad 2: VEE -> Net-(U20-VIN)
- C6 pad 1: Net-(C12-Pad1) -> Net-(C6-Pad1)
- R41 pad 1: Net-(U12-RF-OUT2) -> Net-(U18-RF-OUT1)
- R5 pad 2: GND -> Net-(R5-Pad2)
- R7 pad 2: GND -> Net-(R7-Pad2)
- TP19 pad 1: Net-(U12-RF-OUT1) -> Net-(U18-RF-OUT2)
- U1 pad 7: Net-(C27-Pad1) (its old number) -> Net-(C5-Pad1)
- U1 pad 8: Net-(C27-Pad1) (its old number) -> Net-(C5-Pad1)
- U10 pad 7: Net-(C12-Pad1) -> Net-(C18-Pad1)
- U10 pad 8: Net-(C12-Pad1) -> Net-(C18-Pad1)
- U15 pad 2: VEE -> Net-(U15-VIN)
- U16 pad 2: VEE -> Net-(U16-VIN)
- U18 pad 1: Net-(U12-RF-OUT1) -> Net-(U18-RF-OUT1)
- U18 pad 4: Net-(U12-RF-OUT2) -> Net-(U18-RF-OUT2)
- U19 pad 6: Net-(J1-In) -> Net-(U19-RF-IN)
- U2 pad 7: Net-(C27-Pad1) (its old number) -> Net-(C3-Pad1)
- U2 pad 8: Net-(C27-Pad1) (its old number) -> Net-(C3-Pad1)
- U20 pad 2: VEE -> Net-(U20-VIN)
- U21 pad 7: VDD -> Net-(C53-Pad1)
- U21 pad 8: VDD -> Net-(C53-Pad1)
- U3 pad 7: Net-(C12-Pad1) -> Net-(C6-Pad1)
- U3 pad 8: Net-(C12-Pad1) -> Net-(C6-Pad1)
- U4 pad 7: Net-(C12-Pad1) -> Net-(C4-Pad1)
- U4 pad 8: Net-(C12-Pad1) -> Net-(C4-Pad1)
- U5 pad 7: Net-(C27-Pad1) (its old number) -> Net-(C15-Pad1)
- U5 pad 8: Net-(C27-Pad1) (its old number) -> Net-(C15-Pad1)
- U6 pad 7: Net-(C12-Pad1) -> Net-(C16-Pad1)
- U6 pad 8: Net-(C12-Pad1) -> Net-(C16-Pad1)
- U9 pad 7: Net-(C27-Pad1) (its old number) -> Net-(C17-Pad1)
- U9 pad 8: Net-(C27-Pad1) (its old number) -> Net-(C17-Pad1)
Routing:
- net VDD: track 197.5 -> 413.0 mm, vias 5 -> 12
- net Net-(C12-Pad1): track 136.6 -> 0.00 mm, vias 4 -> 0
- net Net-(C27-Pad1) (its old number): track 136.3 -> 0.00 mm, vias 4 -> 0
- net Net-(U9-SET): track 8.54 -> 59.9 mm, vias 0 -> 1
- net Net-(U10-SET): track 8.54 -> 59.9 mm, vias 0 -> 1
- net VEE: track 191.3 -> 176.3 mm
- net Net-(J1-In): track 18.9 -> 10.5 mm
- net Net-(U18-RF-OUT2): track 0.00 -> 7.96 mm
- net Net-(C3-Pad1): track 0.00 -> 7.78 mm
- net Net-(C4-Pad1): track 0.00 -> 7.62 mm
- net Net-(U12-RF-OUT1): track 6.57 -> 0.00 mm
- net Net-(U19-RF-IN): track 0.00 -> 6.39 mm
- net Net-(C5-Pad1): track 0.00 -> 5.93 mm
- net Net-(C6-Pad1): track 0.00 -> 5.93 mm
- net Net-(C15-Pad1): track 0.00 -> 5.90 mm
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Other:
- board text added: "+5V_CH1"
- board text added: "+5V_CH2"
- board text added: "-5V_CH1"
- board text added: "-5V_CH2"
- board text added: "0V"
- board text added: "2-Tone Acousto-Optic Modulator Driver v2"
- board text added: "5V"
- board text added: "CH 1"
- board text added: "CH 2"
- board text added: "Jacob Feder 2024-2-23"
- board text added: "MHz"
- board text added: "OUT"
- board text added: "VDD_VCO_CH1"
- board text added: "VDD_VCO_CH2"
- board text added: "VVA_TUNE_CH1"
- board text added: "VVA_TUNE_CH2"
- board text removed: "+5V_F1"
- board text removed: "+5V_F2"
- board text removed: "-5V_F1"
- board text removed: "-5V_F2"
- board text removed: "2-Tone Acousto-Optic Modulator Driver v1"
- board text removed: "Jacob Feder 2024-1-1"
- board text removed: "VCO_TUNE_F1"
- board text removed: "VCO_TUNE_F2"
- board text removed: "VDD_VCO_F1"
- board text removed: "VDD_VCO_F2"
- board text removed: "VVA_TUNE_F1"
- board text removed: "VVA_TUNE_F2"
