File: freq_synth.kicad_sch (KiCad schematic)
At the start: 60 parts, among them U1 LT3082xDD, U10 RVA-3000R, U2 LT3082xDD, U3 LT3082xDD, U4 LT3082xDD, U5 PAT1220-C-8DB, U6 GVA-81, U8 ADP7182AUJZ-5.0, U9 M3SWA-2-50, X1 CVCO55xx

Commit message: v2
Parts:
- removed C19: 2.2u, Capacitor_SMD:C_0805_2012Metric_Pad1.18x1.45mm_HandSolder, symbol Device:C
- removed L1, L3: 10u, Inductor_SMD:L_0805_2012Metric_Pad1.05x1.20mm_HandSolder, symbol Device:L
- removed RV1: 2M, Potentiometer_THT:Potentiometer_Bourns_3296Y_Vertical, symbol Device:R_Potentiometer
- added C12, C13, C18, C21, C27: 0.1u, Capacitor_SMD:C_0805_2012Metric_Pad1.18x1.45mm_HandSolder, symbol Device:C
- added R12, R13, R19, R20, R27, R31: 0, Resistor_SMD:R_0805_2012Metric_Pad1.20x1.40mm_HandSolder, symbol Device:R
- added R17, R18, R24, R26: 1.5k, Resistor_SMD:R_0805_2012Metric_Pad1.20x1.40mm_HandSolder, symbol Device:R
- R14: renamed from R1; value 2.7M -> 150k; DKPN 13-RC0805FR-072M7LCT-ND -> 311-150KCRCT-ND; MFPN RC0805FR-072M7L -> RC0805FR-07150KL
- R16: renamed from R4; value 432 -> 4.7k; DKPN 311-432CRCT-ND -> 13-RC0805FR-134K7LCT-ND; MFPN RC0805FR-07432RL -> RC0805FR-134K7L
- R23: renamed from R6; value 432 -> 4.7k; DKPN 311-432CRCT-ND -> 13-RC0805FR-134K7LCT-ND; MFPN RC0805FR-07432RL -> RC0805FR-134K7L
- R30: renamed from R10; value 432 -> 4.7k; DKPN 311-432CRCT-ND -> 13-RC0805FR-134K7LCT-ND; MFPN RC0805FR-07432RL -> RC0805FR-134K7L
- RV1: renamed from RV2; footprint Potentiometer_THT:Potentiometer_Bourns_3296Y_Vertical -> Potentiometer_THT:Potentiometer_Bourns_3296X_Horizontal; DKPN 3296Y-205LF-ND -> 3296X-205LF-ND; MFPN 3296Y-1-205LF -> 3296X-1-205LF
- U11: renamed from U8; DKPN 505-ADP7182ACPZ-5.0-R7CT-ND -> 505-ADP7182AUJZ-5.0-R7CT-ND; MFPN ADP7182ACPZ-5.0-R7 -> ADP7182AUJZ-5.0-R7
- renumbered C2 to C10, C4 to C11, C5 to C14, C6 to C15, C8 to C16, C3 to C17, C9 to C19, C10 to C20, C11 to C22, C12 to C23, C7 to C24, C13 to C25, C15 to C26, C16 to C28, C17 to C29, C18 to C30, C20 to C31, C1 to C9, D1 to D5, D2 to D6, D3 to D7, L2 to L1, R3 to R15, R5 to R21, R2 to R22, R7 to R25, R8 to R28, R9 to R29, R11 to R32, TP2 to TP10, TP7 to TP11, TP8 to TP12, TP9 to TP13, TP8 to TP14, TP10 to TP15, TP1 to TP5, TP3 to TP6, TP4 to TP7, TP5 to TP8, TP6 to TP9, U9 to U12, U1 to U4, U2 to U5, U4 to U6, U5 to U7, U3 to U8, U6 to U9
Connections:
- net +5V: now also R24.1, R31.1
- net GND: now also C12.2, C13.2, C18.2, C21.2, C27.1, R17.2, R18.2, R24.2, R26.2
- net VCO_TUNE: now also R17.1
- net VDD: now also R12.1, R13.1, R19.1, R20.1
- net VDD_VCO: now also R18.1
- net VEE: now also R27.2; no longer C26.2, U11.2 (VIN)
- net VVA_TUNE: now also R26.1
- net at R15.1, U4.4 (SET): now also C13.1
- net at R22.1, RV1.1, U8.4 (SET): now also C21.1
- net at R28.2, R29.2, U11.3 (EN): now also C27.2
- net at R14.1, U5.4 (SET): now also C12.1
- net at C31.1, U12.5 (VDD): now also R31.2
- net at R21.1, U6.4 (SET): now also C18.1
- new net: C26.2, R27.1, U11.2 (VIN)
- new net: C17.1, R20.2, U8.7 (IN), U8.8 (IN)
- new net: C11.1, R13.2, U4.7 (IN), U4.8 (IN)
- new net: C10.1, R12.2, U5.7 (IN), U5.8 (IN)
- new net: C16.1, R19.2, U6.7 (IN), U6.8 (IN)
Other:
- moved on the sheet: C11, C16, C17, C26, C28, C29, C30, C31, C9, D7, FL1, R14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
